File: SC8703_Buck-Boost.kicad_pcb (KiCad board)
At the start: 2 copper layers, 79.6 x 47 mm, 60 parts, among them J1 XT30PW-M, J2 XT30PW-F, J3 USB_C_Receptacle_USB2.0_16P, Q1 XRS100N06LD, Q2 XRS100N06LD, Q3 XRS100N06LD, Q4 XRS100N06LD, U1 SC8703, U2 CH224Q

Commit message: PCB layout 完成5%
Parts:
- moved J3 69.9 mm to (102.7, 81.0), turned to -90 degrees
- moved RV2 54.2 mm to (172.7, 88.0), turned to 180 degrees
- moved C5 6.03 mm to (120.7, 67.4)
- moved J1 6.00 mm to (111.8, 65.0)
Changed lines of the file:
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@@
 	(footprint "Potentiometer_THT:Potentiometer_Bourns_3296X_Horizontal"
 		(layer "F.Cu")
-		(at 127.4636 117.957)
+		(at 172.6692 88 180)
 		(descr "Potentiometer, horizontal, Bourns 3296X, https://www.bourns.com/pdfs/3296.pdf")
 		(tags "Potentiometer horizontal Bourns 3296X")
@@
 		(attr through_hole)
 		(fp_line
-			(start -8.935 -0.055)
-			(end -7.415 -0.055)
+			(start 2.335 2.53)
+			(end -7.415 2.53)
 			(stroke
 				(width 0.12)
@@
 		)
 		(fp_line
-			(start -8.935 1.15)
-			(end -8.175 1.15)
+			(start 2.335 -2.52)
+			(end 2.335 2.53)
 			(stroke
 				(width 0.12)
@@
 		)
 		(fp_line
-			(start -8.935 2.355)
-			(end -8.935 -0.055)
+			(start -7.415 2.53)
+			(end -7.415 -2.52)
 			(stroke
 				(width 0.12)
@@
 		)
 		(fp_line
-			(start -7.415 -2.52)
-			(end 2.335 -2.52)
+			(start -7.415 2.355)
+			(end -8.935 2.355)
 			(stroke
 				(width 0.12)
@@
 		)
 		(fp_line
-			(start -7.415 2.355)
-			(end -8.935 2.355)
+			(start -7.415 -2.52)
+			(end 2.335 -2.52)
 			(stroke
 				(width 0.12)
@@
 		)
 		(fp_line
-			(start -7.415 2.53)
-			(end -7.415 -2.52)
+			(start -8.935 2.355)
+			(end -8.935 -0.055)
 			(stroke
 				(width 0.12)
@@
 		)
 		(fp_line
-			(start 2.335 -2.52)
-			(end 2.335 2.53)
+			(start -8.935 1.15)
+			(end -8.175 1.15)
 			(stroke
 				(width 0.12)
@@
 		)
 		(fp_line
-			(start 2.335 2.53)
-			(end -7.415 2.53)
+			(start -8.935 -0.055)
+			(end -7.415 -0.055)
 			(stroke
 				(width 0.12)
@@
 		)
 		(fp_rect
-			(start -8.825 0.055)
-			(end -7.305 2.245)
+			(start -7.305 -2.41)
+			(end 2.225 2.42)
 			(stroke
 				(width 0.1)
@@
 		)
 		(fp_rect
-			(start -7.305 -2.41)
-			(end 2.225 2.42)
+			(start -8.825 0.055)
+			(end -7.305 2.245)
 			(stroke
 				(width 0.1)
@@
 		)
 		(pad "1" thru_hole circle
-			(at 0 0)
+			(at 0 0 180)
 			(size 1.44 1.44)
 			(drill 0.8)
@@
 		)
 		(pad "2" thru_hole circle
-			(at -2.54 0)
+			(at -2.54 0 180)
 			(size 1.44 1.44)
 			(drill 0.8)
@@
 		)
 		(pad "3" thru_hole circle
-			(at -5.08 0)
+			(at -5.08 0 180)
 			(size 1.44 1.44)
 			(drill 0.8)
@@
 	(footprint "Capacitor_SMD:CP_Elec_10x10.5"
 		(layer "F.Cu")
-		(at 120.1674 73.3825 90)
+		(at 120.7262 67.3825 90)
 		(descr "SMD capacitor, aluminum electrolytic, Vishay 1010, 10.0x10.5mm, http://www.vishay.com/docs/28395/150crz.pdf")
 		(tags "capacitor electrolytic")
@@
 	(footprint "Connector_USB:USB_C_Receptacle_HCTL_HC-TYPE-C-16P-01A"
 		(layer "F.Cu")
-		(at 148.6436 133.647)
+		(at 102.7258 81 -90)
 		(descr "16-pin USB-C receptacle, USB2.0 and PD, 5A VBUS rating, https://datasheet.lcsc.com/lcsc/2211161000_HCTL-HC-TYPE-C-16P-01A_C2894897.pdf")
 		(tags "usb usb-c 2.0 pd")
 		(property "Reference" "J3"
-			(at 0 -5.645 0)
+			(at 0 -5.645 90)
 			(layer "F.SilkS")
 			(hide yes)
@@
 		)
 		(property "Value" "USB_C_Receptacle_USB2.0_16P"
-			(at 0 5 0)
+			(at 0 5 270)
 			(unlocked yes)
 			(layer "F.Fab")
@@
 		)
 		(property "Datasheet" "https://www.usb.org/sites/default/files/documents/usb_type-c.zip"
-			(at 0 0 0)
+			(at 0 0 270)
 			(unlocked yes)
 			(layer "F.Fab")
@@
 		)
 		(property "Description" "USB 2.0-only 16P Type-C Receptacle connector"
-			(at 0 0 0)
+			(at 0 0 270)
 			(unlocked yes)
 			(layer "F.Fab")
@@
 		)
 		(fp_line
-			(start -2.8 -4.7)
-			(end -3.6 -4.7)
+			(start 4.7 -1.78)
+			(end 4.7 0)
 			(stroke
 				(width 0.12)
-				(type default)
+				(type solid)
 			)
 			(layer "F.SilkS")
 		)
 		(fp_line
-			(start 4.7 -1.78)
-			(end 4.7 0)
+			(start -2.8 -4.7)
+			(end -3.6 -4.7)
 			(stroke
 				(width 0.12)
-				(type solid)
+				(type default)
 			)
 			(layer "F.SilkS")
 		)
 		(fp_line
-			(start -0.5 2.5)
+			(start 0 3.5)
 			(end 0 1.5)
 			(stroke
@@
 		)
 		(fp_line
-			(start 0 1.5)
-			(end 0.5 2.5)
+			(start -0.5 2.5)
+			(end 0 1.5)
 			(stroke
 				(width 0.12)
@@
 		)
 		(fp_line
-			(start 0 3.5)
-			(end 0 1.5)
+			(start 0.5 2.5)
+			(end -0.5 2.5)
 			(stroke
 				(width 0.12)
@@
 		)
 		(fp_line
-			(start 0.5 2.5)
-			(end -0.5 2.5)
+			(start 0 1.5)
+			(end 0.5 2.5)
 			(stroke
 				(width 0.12)
@@
 		)
 		(fp_line
-			(start -5.32 -4.9)
-			(end -5.32 4.18)
+			(start -5.32 4.18)
+			(end 5.32 4.18)
 			(stroke
 				(width 0.05)
@@
 		(fp_line
 			(start -5.32 -4.9)
-			(end 5.32 -4.9)
+			(end -5.32 4.18)
 			(stroke
 				(width 0.05)
@@
 		)
 		(fp_line
-			(start -5.32 4.18)
-			(end 5.32 4.18)
+			(start -5.32 -4.9)
+			(end 5.32 -4.9)
 			(stroke
 				(width 0.05)
@@
 		)
 		(fp_line
-			(start -4.47 -3.675)
-			(end -4.47 3.675)
+			(start -4.47 3.675)
+			(end 4.47 3.675)
 			(stroke
 				(width 0.1)
@@
 		)
 		(fp_line
-			(start -4.47 -3.675)
-			(end 4.47 -3.675)
+			(start -3.2 -2.675)
+			(end -4.2 -3.675)
 			(stroke
 				(width 0.1)
-				(type solid)
+				(type default)
 			)
 			(layer "F.Fab")
 		)
 		(fp_line
-			(start -4.47 3.675)
-			(end 4.47 3.675)
+			(start -3.2 -2.675)
+			(end -2.2 -3.675)
 			(stroke
 				(width 0.1)
-				(type solid)
+				(type default)
 			)
 			(layer "F.Fab")
 		)
 		(fp_line
-			(start -3.2 -2.675)
-			(end -4.2 -3.675)
+			(start -4.47 -3.675)
+			(end -4.47 3.675)
 			(stroke
 				(width 0.1)
-				(type default)
+				(type solid)
 			)
 			(layer "F.Fab")
 		)
 		(fp_line
-			(start -3.2 -2.675)
-			(end -2.2 -3.675)
+			(start -4.47 -3.675)
+			(end 4.47 -3.675)
 			(stroke
 				(width 0.1)
-				(type default)
+				(type solid)
 			)
 			(layer "F.Fab")
@@
 		)
 		(fp_text user "${REFERENCE}"
-			(at 0 -0.435 0)
+			(at 0 -0.435 270)
 			(unlocked yes)
 			(layer "F.Fab")
@@
 		)
 		(pad "" np_thru_hole circle
-			(at -2.89 -2.605)
+			(at -2.89 -2.605 270)
 			(size 0.65 0.65)
 			(drill 0.65)
@@
 		)
 		(pad "" np_thru_hole circle
-			(at 2.89 -2.605)
+			(at 2.89 -2.605 270)
 			(size 0.65 0.65)
 			(drill 0.65)
@@
 		)
 		(pad "A1" smd roundrect
-			(at -3.2 -3.745)
+			(at -3.2 -3.745 270)
 			(size 0.6 1.3)
 			(layers "F.Cu" "F.Mask" "F.Paste")
@@
 		)
 		(pad "A4" smd roundrect
-			(at -2.4 -3.745)
+			(at -2.4 -3.745 270)
 			(size 0.6 1.3)
 			(layers "F.Cu" "F.Mask" "F.Paste")
@@
 		)
 		(pad "A5" smd roundrect
-			(at -1.25 -3.745)
+			(at -1.25 -3.745 270)
 			(size 0.3 1.3)
 			(layers "F.Cu" "F.Mask" "F.Paste")
@@
 		)
 		(pad "A6" smd roundrect
-			(at -0.25 -3.745)
+			(at -0.25 -3.745 270)
 			(size 0.3 1.3)
 			(layers "F.Cu" "F.Mask" "F.Paste")
@@
 		)
 		(pad "A7" smd roundrect
-			(at 0.25 -3.745)
+			(at 0.25 -3.745 270)
 			(size 0.3 1.3)
 			(layers "F.Cu" "F.Mask" "F.Paste")
@@
 		)
 		(pad "A8" smd roundrect
-			(at 1.25 -3.745)
+			(at 1.25 -3.745 270)
 			(size 0.3 1.3)
 			(layers "F.Cu" "F.Mask" "F.Paste")
@@
 		)
 		(pad "A9" smd roundrect
-			(at 2.4 -3.745)
+			(at 2.4 -3.745 270)
 			(size 0.6 1.3)
 			(layers "F.Cu" "F.Mask" "F.Paste")
@@
 		)
 		(pad "A12" smd roundrect
-			(at 3.2 -3.745)
+			(at 3.2 -3.745 270)
 			(size 0.6 1.3)
 			(layers "F.Cu" "F.Mask" "F.Paste")
@@
 		)
 		(pad "B1" smd roundrect
-			(at 3.2 -3.745)
+			(at 3.2 -3.745 270)
 			(size 0.6 1.3)
 			(layers "F.Cu" "F.Mask" "F.Paste")
@@
 		)
 		(pad "B4" smd roundrect
-			(at 2.4 -3.745)
+			(at 2.4 -3.745 270)
 			(size 0.6 1.3)
 			(layers "F.Cu" "F.Mask" "F.Paste")
@@
 		)
 		(pad "B5" smd roundrect
-			(at 1.75 -3.745)
+			(at 1.75 -3.745 270)
 			(size 0.3 1.3)
 			(layers "F.Cu" "F.Mask" "F.Paste")
@@
 		)
 		(pad "B6" smd roundrect
-			(at 0.75 -3.745)
+			(at 0.75 -3.745 270)
 			(size 0.3 1.3)
 			(layers "F.Cu" "F.Mask" "F.Paste")
@@
 		)
 		(pad "B7" smd roundrect
-			(at -0.75 -3.745)
+			(at -0.75 -3.745 270)
 			(size 0.3 1.3)
 			(layers "F.Cu" "F.Mask" "F.Paste")
@@
 		)
 		(pad "B8" smd roundrect
-			(at -1.75 -3.745)
+			(at -1.75 -3.745 270)
 			(size 0.3 1.3)
 			(layers "F.Cu" "F.Mask" "F.Paste")
@@
 		)
 		(pad "B9" smd roundrect
-			(at -2.4 -3.745)
+			(at -2.4 -3.745 270)
 			(size 0.6 1.3)
 			(layers "F.Cu" "F.Mask" "F.Paste")
@@
 		)
 		(pad "B12" smd roundrect
-			(at -3.2 -3.745)
+			(at -3.2 -3.745 270)
 			(size 0.6 1.3)
 			(layers "F.Cu" "F.Mask" "F.Paste")
@@
 		)
 		(pad "S1" thru_hole oval
-			(at -4.32 -3.105)
+			(at -4.32 -3.105 270)
 			(size 1 2.1)
 			(drill oval 0.6 1.7)
@@
 		)
 		(pad "S1" thru_hole oval
-			(at -4.32 1.075)
+			(at -4.32 1.075 270)
 			(size 1 1.6)
 			(drill oval 0.6 1.2)
@@
 		)
 		(pad "S1" thru_hole oval
-			(at 4.32 -3.105)
+			(at 4.32 -3.105 270)
 			(size 1 2.1)
 			(drill oval 0.6 1.7)
@@
 		)
 		(pad "S1" thru_hole oval
-			(at 4.32 1.075)
+			(at 4.32 1.075 270)
 			(size 1 1.6)
 			(drill oval 0.6 1.2)
@@
 	(footprint "Connector_AMASS:AMASS_XT30PW-M_1x02_P2.50mm_Horizontal"
 		(layer "F.Cu")
-		(at 111.6946 71 90)
+		(at 111.7962 65 90)
 		(descr "Connector XT30 Horizontal PCB Male, https://www.tme.eu/Document/6eb2005a51a52592b3f19e8a450c54c8/XT30PW-M.pdf")
 		(tags "RC Connector XT30")

Commit message: 修正输出电容数值
Parts:
- C10: value 330uF -> 220uF
Changed lines of the file:
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@@
 			)
 		)
-		(property "Value" "330uF"
+		(property "Value" "220uF"
 			(at 0 6.3 0)
 			(layer "F.Fab")
