File: SC8703_Buck-Boost.kicad_pcb (KiCad board)
At the start: 2 copper layers, 79.6 x 47 mm, 60 parts, among them J1 XT30PW-M, J2 XT30PW-F, J3 USB_C_Receptacle_USB2.0_16P, Q1 XRS100N06LD, Q2 XRS100N06LD, Q3 XRS100N06LD, Q4 XRS100N06LD, U1 SC8703, U2 CH224Q

Commit message: PCB完成95%
Parts:
- added C24: 220uF, Capacitor_SMD:CP_Elec_10x10.5, F.Cu at (130.8, 67.4)
- added C25: 220uF, Capacitor_SMD:CP_Elec_10x10.5, F.Cu at (154.3, 77.4)
- C1, C11, C12, C13, C14, C2, C6, C7, C8, C9, D2, D3, Q1, Q2, Q3, Q4, R1, R10, R11, R12, R13, R14, R2, R7, R8, R9: moved to B.Cu
- moved R14 85.4 mm to (147.3, 56.6), turned to 90 degrees
- moved C13 81.2 mm to (159.6, 63.7), turned to 90 degrees
- moved R10 80.9 mm to (152.2, 56.6), turned to 90 degrees
- moved R8 80.3 mm to (157.2, 63.7), turned to -90 degrees
- moved C12 78.8 mm to (162.0, 63.7), turned to 90 degrees
- moved R13 73.6 mm to (143.0, 65.6), turned to 90 degrees
- moved C9 73.1 mm to (131.0, 64.5), turned to -90 degrees
- moved C23 71.5 mm to (113.9, 80.7), turned to 180 degrees
- moved R7 71.5 mm to (132.8, 63.7), turned to 90 degrees
- moved C11 70.1 mm to (155.6, 67.5), turned to 180 degrees
- moved R1 69.9 mm to (136.9, 59.4)
- moved C14 69.0 mm to (170.0, 67.5), turned to -90 degrees
- moved R9 68.6 mm to (137.8, 65.6), turned to 90 degrees
- moved C8 68.4 mm to (124.4, 63.7), turned to 90 degrees
- moved R2 67.4 mm to (151.0, 65.0)
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Routing:
- net VOUT: track 0.00 -> 81.6 mm, vias 0 -> 25
- net VIN: track 0.00 -> 45.5 mm, vias 0 -> 19
- net /FB: track 0.00 -> 43.7 mm
- net /HD2: track 0.00 -> 42.5 mm, vias 0 -> 1
- net Net-(Q2-D): track 0.00 -> 33.3 mm, vias 0 -> 1
- net /LD2: track 0.00 -> 32.5 mm, vias 0 -> 1
- net /SW2: track 0.00 -> 28.5 mm, vias 0 -> 15
- net /SW1: track 0.00 -> 22.7 mm, vias 0 -> 15
- net /LD1: track 0.00 -> 19.8 mm, vias 0 -> 1
- net /CC1: track 0.00 -> 18.1 mm, vias 0 -> 2
- net /HD1: track 0.00 -> 17.4 mm, vias 0 -> 1
- net VCC: track 0.00 -> 16.6 mm, vias 0 -> 2
- net Net-(Q1-D): track 0.00 -> 16.2 mm, vias 0 -> 1
- net GND: track 0.00 -> 15.3 mm, vias 0 -> 198
- net Net-(R18-Pad1): track 0.00 -> 14.2 mm
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- added copper zone on B.Cu, net /SW1
- added copper zone on F.Cu, net /SW1
- added copper zone on B.Cu, net /SW2
- added copper zone on F.Cu, net /SW2
- added copper zone on F.Cu, net /VBUS
- added copper zone on B.Cu, net GND
- added copper zone on F.Cu, net GND
- added copper zone on B.Cu, net Net-(Q1-D)
- added copper zone on B.Cu, net Net-(Q2-D)
- added copper zone on B.Cu, net VIN
- added copper zone on F.Cu, net VIN
- added copper zone on B.Cu, net VOUT
- added copper zone on F.Cu, net VOUT
Other:
- outline, holes or cut-outs redrawn
- board text added: "IN"
- board text added: "OUT"

Commit message: 设计完成，下单打样
Parts:
- added G***: LOGO, LOGO, F.Cu at (123.3, 89.6)
- added G***: LOGO, LOGO, B.Cu at (123.2, 89.6)
- RV1: footprint Potentiometer_THT:Potentiometer_Bourns_3296W_Vertical -> Potentiometer_THT:Potentiometer_Bourns_3296X_Horizontal
- moved RV1 46.2 mm to (171.9, 86.5), turned to 180 degrees
Connections:
- RV1 pad 1: Net-(R18-Pad1) -> GND
- RV1 pad 3: GND -> Net-(R18-Pad1)
Routing:
- net Net-(R18-Pad1): track 14.2 -> 47.4 mm
Other:
- board text added: "JLCJLCJLCJLC"
- board text added: "SC8703 Buck-Boost 升降压DCDC"
- board text added: "V1.0"
- board text added: "https://blog.zeruns.com"
- board text added: "电压"
- board text added: "电流"
- board text added: "输入电压：2.7-36V 输出电压：2.5-36V 最大电流：10.2A"
